Commit message: changed slam package

File: src/maddrone/urdf/maddrone.urdf (robot description, URDF)
Before this commit: robot Starling2, 16 links, 15 joints
Joints:
- joint tof_to_tof_pc: origin xyz=0 0 0 rpy=3.141592653589793 1.5707963267948966 3.141592653589793 -> xyz=0 0 0 rpy=1.5707963267948966 1.5707963267948966 1.5707963267948966
